Commit message: basic_convert

File: assets/robot/urdf/uni_dingo_lite.urdf (robot description, URDF)
Before this commit: robot uni_dingo_lite, 22 links, 21 joints
Links:
- link base_link: geometry visual box size=0.001 0.001 0.001
- link left_gripperMover: geometry collision mesh filename=package://z1_description/meshes/collision/z1_GripperMover.S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 scale=1 1 1; visual mesh filename=package://z1_description/meshes/visual/z1_GripperMover.dae scale=1 1 1
- link left_gripperStator: geometry collision mesh filename=package://z1_description/meshes/collision/z1_GripperStator.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 scale=1 1 1; visual mesh filename=package://z1_description/meshes/visual/z1_GripperStator.dae scale=1 1 1
- link left_link00: geometry collision cylinder length=0.051 radius=0.0325; visual mesh filename=package://z1_description/meshes/visual/z1_Link00.dae scale=1 1 1
- link left_link01: geometry collision mesh filename=package://z1_description/meshes/collision/z1_Link01.STL scale=1 1 1; visual mesh filename=package://z1_description/meshes/visual/z1_Link01.dae scale=1 1 1
- link left_link02: geometry collision cylinder length=0.102 radius=0.0325; visual mesh filename=package://z1_description/meshes/visual/z1_Link02.dae scale=1 1 1
- link left_link03: geometry collision cylinder length=0.116 radius=0.02; visual mesh filename=package://z1_description/meshes/visual/z1_Link03.dae scale=1 1 1
- link left_link04: geometry collision cylinder length=0.067 radius=0.0325; visual mesh filename=package://z1_description/meshes/visual/z1_Link04.dae scale=1 1 1
- link left_link05: geometry collision mesh filename=package://z1_description/meshes/collision/z1_Link05.STL scale=1 1 1; visual mesh filename=package://z1_description/meshes/visual/z1_Link05.dae scale=1 1 1
- link left_link06: geometry collision cylinder length=0.051 radius=0.0325; visual mesh filename=package://z1_description/meshes/visual/z1_Link06.dae scale=1 1 1
- link leftarm_link: geometry collision cylinder length=0.47228 radius=0.02; visual cylinder length=0.47228 radius=0.02
- link right_gripperMover: geometry collision mesh filename=package://z1_description/meshes/collision/z1_GripperMover.S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 scale=1 1 1; visual mesh filename=package://z1_description/meshes/visual/z1_GripperMover.dae scale=1 1 1
- link right_gripperStator: geometry collision mesh filename=package://z1_description/meshes/collision/z1_GripperStator.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 scale=1 1 1; visual mesh filename=package://z1_description/meshes/visual/z1_GripperStator.dae scale=1 1 1
- link right_link00: geometry collision cylinder length=0.051 radius=0.0325; visual mesh filename=package://z1_description/meshes/visual/z1_Link00.dae scale=1 1 1
- link right_link01: geometry collision mesh filename=package://z1_description/meshes/collision/z1_Link01.STL scale=1 1 1; visual mesh filename=package://z1_description/meshes/visual/z1_Link01.dae scale=1 1 1
- link right_link02: geometry collision cylinder length=0.102 radius=0.0325; visual mesh filename=package://z1_description/meshes/visual/z1_Link02.dae scale=1 1 1
- link right_link03: geometry collision cylinder length=0.116 radius=0.02; visual mesh filename=package://z1_description/meshes/visual/z1_Link03.dae scale=1 1 1
- link right_link04: geometry collision cylinder length=0.067 radius=0.0325; visual mesh filename=package://z1_description/meshes/visual/z1_Link04.dae scale=1 1 1
- link right_link05: geometry collision mesh filename=package://z1_description/meshes/collision/z1_Link05.STL scale=1 1 1; visual mesh filename=package://z1_description/meshes/visual/z1_Link05.dae scale=1 1 1
- link right_link06: geometry collision cylinder length=0.051 radius=0.0325; visual mesh filename=package://z1_description/meshes/visual/z1_Link06.dae scale=1 1 1
- link rightarm_link: geometry collision cylinder length=0.47228 radius=0.02; visual cylinder length=0.47228 radius=0.02

Commit message: 碰撞体积修改

File: assets/robot/urdf/uni_dingo_lite.urdf (robot description, URDF)
Before this commit: robot uni_dingo_lite, 22 links, 21 joints
Links:
- link left_link00: geometry collision mesh filename=package://z1_description/meshes/collision/z1_Link00.STL scale=1 1 1; visual mesh filename=package://z1_description/meshes/visual/z1_Link00.dae scale=1 1 1
- link left_link02: geometry collision mesh filename=package://z1_description/meshes/collision/z1_Link02.STL scale=1 1 1; visual mesh filename=package://z1_description/meshes/visual/z1_Link02.dae scale=1 1 1
- link left_link03: geometry collision mesh filename=package://z1_description/meshes/collision/z1_Link03.STL scale=1 1 1; visual mesh filename=package://z1_description/meshes/visual/z1_Link03.dae scale=1 1 1
- link left_link04: geometry collision mesh filename=package://z1_description/meshes/collision/z1_Link04.STL scale=1 1 1; visual mesh filename=package://z1_description/meshes/visual/z1_Link04.dae scale=1 1 1
- link left_link06: geometry collision mesh filename=package://z1_description/meshes/collision/z1_Link06.STL scale=1 1 1; visual mesh filename=package://z1_description/meshes/visual/z1_Link06.dae scale=1 1 1
- link right_link00: geometry collision mesh filename=package://z1_description/meshes/collision/z1_Link00.STL scale=1 1 1; visual mesh filename=package://z1_description/meshes/visual/z1_Link00.dae scale=1 1 1
- link right_link02: geometry collision mesh filename=package://z1_description/meshes/collision/z1_Link02.STL scale=1 1 1; visual mesh filename=package://z1_description/meshes/visual/z1_Link02.dae scale=1 1 1
- link right_link03: geometry collision mesh filename=package://z1_description/meshes/collision/z1_Link03.STL scale=1 1 1; visual mesh filename=package://z1_description/meshes/visual/z1_Link03.dae scale=1 1 1
- link right_link04: geometry collision mesh filename=package://z1_description/meshes/collision/z1_Link04.STL scale=1 1 1; visual mesh filename=package://z1_description/meshes/visual/z1_Link04.dae scale=1 1 1
- link right_link06: geometry collision mesh filename=package://z1_description/meshes/collision/z1_Link06.STL scale=1 1 1; visual mesh filename=package://z1_description/meshes/visual/z1_Link06.dae scale=1 1 1

Commit message: 加入底盘

File: assets/robot/urdf/uni_dingo_lite.urdf (robot description, URDF)
Before this commit: robot uni_dingo_lite, 22 links, 21 joints
Links:
- added link front_left_wheel_link, mass 0.4; collision cylinder length=0.050 radius=0.050; visual cylinder length=0.050 radius=0.050
- added link front_right_wheel_link, mass 0.4; collision cylinder length=0.050 radius=0.050; visual cylinder length=0.050 radius=0.050
- added link rear_left_wheel_link, mass 0.4; collision cylinder length=0.050 radius=0.050; visual cylinder length=0.050 radius=0.050
- added link rear_right_wheel_link, mass 0.4; collision cylinder length=0.050 radius=0.050; visual cylinder length=0.050 radius=0.050
- link chassis_link: geometry collision mesh filename=package://dingo_description/meshes/omni_chassis_collision.s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; visual mesh filename=package://dingo_description/meshes/omni_chassis.dae
Joints:
- added joint front_left_wheel: type continuous, parent chassis_link, child front_left_wheel_link, origin xyz=0.285 0.2104 0.035145 rpy=0 0 0, axis 0 1 0
- added joint front_right_wheel: type continuous, parent chassis_link, child front_right_wheel_link, origin xyz=0.285 -0.2104 0.035145 rpy=0 0 0, axis 0 1 0
- added joint rear_left_wheel: type continuous, parent chassis_link, child rear_left_wheel_link, origin xyz=-0.285 0.2104 0.035145 rpy=0 0 0, axis 0 1 0
- added joint rear_right_wheel: type continuous, parent chassis_link, child rear_right_wheel_link, origin xyz=-0.285 -0.2104 0.035145 rpy=0 0 0, axis 0 1 0

Commit message: 底盘可加入训练

File: assets/robot/urdf/uni_dingo_lite.urdf (robot description, URDF)
Before this commit: robot uni_dingo_lite, 26 links, 25 joints
Links:
- added link base_x_link, mass 0.001
- added link base_y_link, mass 0.001
- added link planar_base_root_link, mass 0.001
Joints:
- added joint base_x_joint: type prismatic, parent planar_base_root_link, child base_x_link, origin xyz=0 0 0 rpy=0 0 0, axis 1 0 0, limit lower=-20.0 upper=20.0 effort=1000000.0 velocity=10.0
- added joint base_y_joint: type prismatic, parent base_x_link, child base_y_link, origin xyz=0 0 0 rpy=0 0 0, axis 0 1 0, limit lower=-20.0 upper=20.0 effort=1000000.0 velocity=10.0
- added joint base_yaw_joint: type continuous, parent base_y_link, child base_link, origin xyz=0 0 0.014855 rpy=0 0 0, axis 0 0 1
